File: Rover_Commander_v3.1a.sch (KiCad schematic (older format))
At the start: 75 parts, among them Q1 Crystal KX-7 25MHz, Q2 Crystal KX-7 25MHz, U1 RTL8201CP, U2 L7805ABD2T-TR, U3 H1102NLT, U4 LD1117S33TR_SOT223, U5 STM32F107RCTx, U6 TJA1040T, U7 M95160-WMN6TP

Commit message: fix ICs libs, add .sh jobs, plot .sch to .png & .pdf
Parts:
- U5: symbol STM32F107RCTx-RESCUE-Rover_Commander_v3.1a -> STM32F107RCTx
Changed lines of the file:
@@
 EESchema Schematic File Version 2
-LIBS:Rover_Commander_v3.1a-rescue
 LIBS:power
 LIBS:device
@@
 LIBS:M95160-WMN6TP
 LIBS:L7805ABD2T-TR
+LIBS:tja1040t
+LIBS:RTL8201CP
+LIBS:h1102nlt
 LIBS:Rover_Commander_v3.1a-cache
 EELAYER 25 0
@@
 $EndDescr
 $Comp
-L STM32F107RCTx-RESCUE-Rover_Commander_v3.1a U5
+L STM32F107RCTx U5
 U 1 1 59D8B1C8
 P 10300 3700
@@
 $EndComp
 $Comp
-L TJA1040T U6
-U 1 1 59DE414E
-P 14200 6450
-F 0 "U6" H 13800 6800 50  0000 L CNN
-F 1 "TJA1040T" H 14250 6800 50  0000 L CNN
-F 2 "Housings_SOIC:SOIC-8_3.9x4.9mm_Pitch1.27mm" H 14200 5950 50  0001 C CIN
-F 3 "" H 14200 6450 50  0001 C CNN
-	1    14200 6450
-	1    0    0    -1
-$EndComp
-$Comp
 L R R19
 U 1 1 59DE54C8
@@
 	4500 6900 4500 6750
 Connection ~ 4500 6900
+$Comp
+L TJA1040T U6
+U 1 1 5A82C7AF
+P 14200 6450
+F 0 "U6" H 13800 6800 50  0000 L CNN
+F 1 "TJA1040T" H 14250 6800 50  0000 L CNN
+F 2 "Housings_SOIC:SOIC-8_3.9x4.9mm_Pitch1.27mm" H 14200 5950 50  0001 C CIN
+F 3 "" H 14200 6450 50  0001 C CNN
+	1    14200 6450
+	1    0    0    -1
+$EndComp
 $EndSCHEMATC
